Commit message: updated urdf, robot in gazebo

File: pff_rohit/urdf/diff_drive.urdf (robot description, URDF)
Before this commit: robot diff_drive_robot, 4 links, 3 joints
Links:
- link body: mass None -> 10; geometry collision box size=0.1 0.1 0.05; visual box size=0.1 0.1 0.05
- link head: mass None -> 5; geometry collision box size=0.05 0.05 0.04; visual box size=0.05 0.05 .04
- link wheel_left: mass None -> 3; geometry collision cylinder length=0.02 radius=0.04; visual cylinder length=0.02 radius=0.04
- link wheel_right: mass None -> 3; geometry collision cylinder length=0.02 radius=0.04; visual cylinder length=0.02 radius=0.04

Commit message: a more complete urdf

File: pff_rohit/urdf/diff_drive.urdf (robot description, URDF)
Before this commit: robot diff_drive_robot, 4 links, 3 joints
Joints:
- joint body_to_left_wheel: limit (none) -> effort=100 velocity=100
- joint body_to_right_wheel: limit (none) -> effort=100 velocity=100

Commit message: cmd_vel publisher

File: pff_rohit/urdf/diff_drive.urdf (robot description, URDF)
Before this commit: robot diff_drive_robot, 4 links, 3 joints
Joints:
- joint body_to_head: origin xyz=0.075 0 0.04 rpy=0 0 0 -> xyz=0.075 0 0.02 rpy=0 0 0
- joint body_to_left_wheel: axis 0 1 0 -> 0 0 -1; origin xyz=0 0.06 0.04 rpy=1.57075 0 0 -> xyz=0 0.06 0.02 rpy=1.57075 0 0
- joint body_to_right_wheel: axis 0 -1 0 -> 0 0 -1; origin xyz=0 -0.06 0.04 rpy=1.57075 0 0 -> xyz=0 -0.06 0.02 rpy=1.57075 0 0

Commit message: robot moves using teleop, to add: Caster Wheel and Improve keypad movement

File: pff_rohit/urdf/diff_drive.urdf (robot description, URDF)
Before this commit: robot diff_drive_robot, 4 links, 3 joints
Links:
- link head: mass 5 -> 1

Commit message: moving robot with keys

File: pff_rohit/urdf/diff_drive.urdf (robot description, URDF)
Before this commit: robot diff_drive_robot, 4 links, 3 joints
Links:
- added link caster_wheel_b, mass 4; collision sphere radius=0.01; visual sphere radius=0.01
- added link caster_wheel_f, mass 1; collision sphere radius=0.02; visual sphere radius=0.02
- link body: mass 10 -> 5
- link head: mass 1 -> 2
- link wheel_left: mass 3 -> 6
- link wheel_right: mass 3 -> 6
Joints:
- added joint caster_back_joint: type fixed, parent body, child caster_wheel_b, origin xyz=-0.02 0.0 -0.01 rpy=0 0 0
- added joint caster_front_joint: type fixed, parent head, child caster_wheel_f, origin xyz=0.0 0.0 -0.02 rpy=0 0 0

Commit message: improved motion of the robot and updated urdf with proper inertias

File: pff_rohit/urdf/diff_drive.urdf (robot description, URDF)
Before this commit: robot diff_drive_robot, 6 links, 5 joints
Links:
- link body: mass 5 -> 3
- link caster_wheel_b: mass 4 -> 1
- link wheel_left: mass 6 -> 2.5
- link wheel_right: mass 6 -> 2.5
Joints:
- joint body_to_left_wheel: limit effort=100 velocity=100 -> effort=1000 velocity=1000
- joint body_to_right_wheel: limit effort=100 velocity=100 -> effort=1000 velocity=1000
